File: 05_CONTROL-ELECTRONICS/TREC/MCU.kicad_sch (KiCad schematic)
At the start: 17 parts, among them J1 USB_B_Micro, J2 Conn_01x04_Pin, SW1 SW_SPDT, U1 STM32F401RETx, Y1 16MHz

Commit message: Old kicad changes and BLDC CAD
Other:
- company: (none) -> B Watt
- title: (none) -> MCU Electrical Schematic
Changed lines of the file:
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@@
 	(generator_version "8.0")
 	(paper "A4")
+	(title_block
+		(title "MCU Electrical Schematic")
+		(date "2025-04-20")
+		(rev "0")
+		(company "B Watt")
+	)
 	(junction
 		(at 83.82 21.59)
